File: clock_logics/_autosave-clock_logics.kicad_sch (KiCad schematic)
At the start: 66 parts, among them J1 Conn_01x04_Male, J2 Conn_01x04_Male, J3 Conn_01x04_Male, SW1 SW_DIP_x10, U1 NE555P, U10 4017, U2 NE555P, U3 NE555P, U4 NE555P, U5 4011, U6 4001, U7 74HC240, U8 4020, U9 4076

Commit message: new schematics
Parts:
- J1, J2, J3: footprint Connector_PinSocket_2.54mm:PinSocket_1x04_P2.54mm_Vertical -> Connector_PinSocket_2.54mm:PinSocket_1x04_P2.54mm_Horizontal
- RV1, RV2, RV3, RV4, RV5, RV6, RV7, RV8: footprint Potentiometer_THT:Potentiometer_Runtron_RM-065_Vertical -> Potentiometer_THT:Potentiometer_Piher_PT-6-H_Horizontal
- SW1: footprint Button_Switch_THT:SW_DIP_SPSTx10_Slide_9.78x27.58mm_W7.62mm_P2.54mm -> Button_Switch_THT:SW_DIP_SPSTx10_Piano_10.8x26.96mm_W7.62mm_P2.54mm
Changed lines of the file:
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@@
     (property "Reference" "J1" (id 0) (at 121.285 17.78 0))
     (property "Value" "Conn_01x04_Male" (id 1) (at 121.285 20.32 0))
-    (property "Footprint" "Connector_PinSocket_2.54mm:PinSocket_1x04_P2.54mm_Vertical" (id 2) (at 121.92 25.4 0)
+    (property "Footprint" "Connector_PinSocket_2.54mm:PinSocket_1x04_P2.54mm_Horizontal" (id 2) (at 121.92 25.4 0)
       (effects (font (size 1.27 1.27)) hide)
     )
@@
       (effects (font (size 1.27 1.27)) (justify right))
     )
-    (property "Footprint" "Potentiometer_THT:Potentiometer_Runtron_RM-065_Vertical" (id 2) (at 67.31 250.19 0)
+    (property "Footprint" "Potentiometer_THT:Potentiometer_Piher_PT-6-H_Horizontal" (id 2) (at 67.31 250.19 0)
       (effects (font (size 1.27 1.27)) hide)
     )
@@
       (effects (font (size 1.27 1.27)) (justify right))
     )
-    (property "Footprint" "Potentiometer_THT:Potentiometer_Runtron_RM-065_Vertical" (id 2) (at 67.31 116.84 0)
+    (property "Footprint" "Potentiometer_THT:Potentiometer_Piher_PT-6-H_Horizontal" (id 2) (at 67.31 116.84 0)
       (effects (font (size 1.27 1.27)) hide)
     )
@@
       (effects (font (size 1.27 1.27)) (justify right))
     )
-    (property "Footprint" "Potentiometer_THT:Potentiometer_Runtron_RM-065_Vertical" (id 2) (at 74.93 184.15 0)
+    (property "Footprint" "Potentiometer_THT:Potentiometer_Piher_PT-6-H_Horizontal" (id 2) (at 74.93 184.15 0)
       (effects (font (size 1.27 1.27)) hide)
     )
@@
       (effects (font (size 1.27 1.27)) (justify right))
     )
-    (property "Footprint" "Potentiometer_THT:Potentiometer_Runtron_RM-065_Vertical" (id 2) (at 73.66 58.42 0)
+    (property "Footprint" "Potentiometer_THT:Potentiometer_Piher_PT-6-H_Horizontal" (id 2) (at 73.66 58.42 0)
       (effects (font (size 1.27 1.27)) hide)
     )
@@
     (property "Reference" "J3" (id 0) (at 278.765 173.99 0))
     (property "Value" "Conn_01x04_Male" (id 1) (at 278.765 176.53 0))
-    (property "Footprint" "Connector_PinSocket_2.54mm:PinSocket_1x04_P2.54mm_Vertical" (id 2) (at 279.4 181.61 0)
+    (property "Footprint" "Connector_PinSocket_2.54mm:PinSocket_1x04_P2.54mm_Horizontal" (id 2) (at 279.4 181.61 0)
       (effects (font (size 1.27 1.27)) hide)
     )
@@
       (effects (font (size 1.27 1.27)) (justify right))
     )
-    (property "Footprint" "Potentiometer_THT:Potentiometer_Runtron_RM-065_Vertical" (id 2) (at 67.31 181.61 0)
+    (property "Footprint" "Potentiometer_THT:Potentiometer_Piher_PT-6-H_Horizontal" (id 2) (at 67.31 181.61 0)
       (effects (font (size 1.27 1.27)) hide)
     )
@@
     (property "Reference" "J2" (id 0) (at 234.315 173.99 0))
     (property "Value" "Conn_01x04_Male" (id 1) (at 234.315 176.53 0))
-    (property "Footprint" "Connector_PinSocket_2.54mm:PinSocket_1x04_P2.54mm_Vertical" (id 2) (at 233.68 181.61 0)
+    (property "Footprint" "Connector_PinSocket_2.54mm:PinSocket_1x04_P2.54mm_Horizontal" (id 2) (at 233.68 181.61 0)
       (effects (font (size 1.27 1.27)) hide)
     )
@@
     (property "Reference" "SW1" (id 0) (at 133.35 43.18 0))
     (property "Value" "SW_DIP_x10" (id 1) (at 133.35 45.72 0))
-    (property "Footprint" "Button_Switch_THT:SW_DIP_SPSTx10_Slide_9.78x27.58mm_W7.62mm_P2.54mm" (id 2) (at 133.35 63.5 0)
+    (property "Footprint" "Button_Switch_THT:SW_DIP_SPSTx10_Piano_10.8x26.96mm_W7.62mm_P2.54mm" (id 2) (at 133.35 63.5 0)
       (effects (font (size 1.27 1.27)) hide)
     )
@@
       (effects (font (size 1.27 1.27)) (justify right))
     )
-    (property "Footprint" "Potentiometer_THT:Potentiometer_Runtron_RM-065_Vertical" (id 2) (at 74.93 119.38 0)
+    (property "Footprint" "Potentiometer_THT:Potentiometer_Piher_PT-6-H_Horizontal" (id 2) (at 74.93 119.38 0)
       (effects (font (size 1.27 1.27)) hide)
     )
@@
       (effects (font (size 1.27 1.27)) (justify right))
     )
-    (property "Footprint" "Potentiometer_THT:Potentiometer_Runtron_RM-065_Vertical" (id 2) (at 74.93 252.73 0)
+    (property "Footprint" "Potentiometer_THT:Potentiometer_Piher_PT-6-H_Horizontal" (id 2) (at 74.93 252.73 0)
       (effects (font (size 1.27 1.27)) hide)
     )
@@
       (effects (font (size 1.27 1.27)) (justify right))
     )
-    (property "Footprint" "Potentiometer_THT:Potentiometer_Runtron_RM-065_Vertical" (id 2) (at 66.04 55.88 0)
+    (property "Footprint" "Potentiometer_THT:Potentiometer_Piher_PT-6-H_Horizontal" (id 2) (at 66.04 55.88 0)
       (effects (font (size 1.27 1.27)) hide)
     )
@@
     )
     (path "/131939a9-acb6-4907-8b43-df51f80d4e89"
-      (reference "J1") (unit 1) (value "Conn_01x04_Male") (footprint "Connector_PinSocket_2.54mm:PinSocket_1x04_P2.54mm_Vertical")
+      (reference "J1") (unit 1) (value "Conn_01x04_Male") (footprint "Connector_PinSocket_2.54mm:PinSocket_1x04_P2.54mm_Horizontal")
     )
     (path "/b792e561-b364-4441-a987-a111d35fbb0a"
-      (reference "J2") (unit 1) (value "Conn_01x04_Male") (footprint "Connector_PinSocket_2.54mm:PinSocket_1x04_P2.54mm_Vertical")
+      (reference "J2") (unit 1) (value "Conn_01x04_Male") (footprint "Connector_PinSocket_2.54mm:PinSocket_1x04_P2.54mm_Horizontal")
     )
     (path "/9d4ac0bc-144a-4f32-8029-59dc8914d1af"
-      (reference "J3") (unit 1) (value "Conn_01x04_Male") (footprint "Connector_PinSocket_2.54mm:PinSocket_1x04_P2.54mm_Vertical")
+      (reference "J3") (unit 1) (value "Conn_01x04_Male") (footprint "Connector_PinSocket_2.54mm:PinSocket_1x04_P2.54mm_Horizontal")
     )
     (path "/c60b8566-48da-4b70-9b22-f29f719c20d0"
@@
     )
     (path "/fac64b7f-351a-4f14-8e09-6c6a4cb59576"
-      (reference "RV1") (unit 1) (value "R_Potentiometer") (footprint "Potentiometer_THT:Potentiometer_Runtron_RM-065_Vertical")
+      (reference "RV1") (unit 1) (value "R_Potentiometer") (footprint "Potentiometer_THT:Potentiometer_Piher_PT-6-H_Horizontal")
     )
     (path "/98926b9b-cc38-4320-bbed-fc5769c45dbc"
-      (reference "RV2") (unit 1) (value "R_Potentiometer") (footprint "Potentiometer_THT:Potentiometer_Runtron_RM-065_Vertical")
+      (reference "RV2") (unit 1) (value "R_Potentiometer") (footprint "Potentiometer_THT:Potentiometer_Piher_PT-6-H_Horizontal")
     )
     (path "/46efad9d-d1cb-4d7c-a051-3ef418d58b89"
-      (reference "RV3") (unit 1) (value "R_Potentiometer") (footprint "Potentiometer_THT:Potentiometer_Runtron_RM-065_Vertical")
+      (reference "RV3") (unit 1) (value "R_Potentiometer") (footprint "Potentiometer_THT:Potentiometer_Piher_PT-6-H_Horizontal")
     )
     (path "/e3a39ab5-bdf2-4067-9ff1-bce139055996"
-      (reference "RV4") (unit 1) (value "R_Potentiometer") (footprint "Potentiometer_THT:Potentiometer_Runtron_RM-065_Vertical")
+      (reference "RV4") (unit 1) (value "R_Potentiometer") (footprint "Potentiometer_THT:Potentiometer_Piher_PT-6-H_Horizontal")
     )
     (path "/aeb1c33f-fe91-439a-a505-a804fd95b515"
-      (reference "RV5") (unit 1) (value "R_Potentiometer") (footprint "Potentiometer_THT:Potentiometer_Runtron_RM-065_Vertical")
+      (reference "RV5") (unit 1) (value "R_Potentiometer") (footprint "Potentiometer_THT:Potentiometer_Piher_PT-6-H_Horizontal")
     )
     (path "/47389f10-669f-4af6-9900-7ad72bad760a"
-      (reference "RV6") (unit 1) (value "R_Potentiometer") (footprint "Potentiometer_THT:Potentiometer_Runtron_RM-065_Vertical")
+      (reference "RV6") (unit 1) (value "R_Potentiometer") (footprint "Potentiometer_THT:Potentiometer_Piher_PT-6-H_Horizontal")
     )
     (path "/1b589a8b-ee14-4199-8a39-c982eda63248"
-      (reference "RV7") (unit 1) (value "R_Potentiometer") (footprint "Potentiometer_THT:Potentiometer_Runtron_RM-065_Vertical")
+      (reference "RV7") (unit 1) (value "R_Potentiometer") (footprint "Potentiometer_THT:Potentiometer_Piher_PT-6-H_Horizontal")
     )
     (path "/f263691f-b3ff-4725-8d8b-47346b209933"
-      (reference "RV8") (unit 1) (value "R_Potentiometer") (footprint "Potentiometer_THT:Potentiometer_Runtron_RM-065_Vertical")
+      (reference "RV8") (unit 1) (value "R_Potentiometer") (footprint "Potentiometer_THT:Potentiometer_Piher_PT-6-H_Horizontal")
     )
     (path "/c49aff7f-db4a-4a23-aa0c-2bfc23209d11"
-      (reference "SW1") (unit 1) (value "SW_DIP_x10") (footprint "Button_Switch_THT:SW_DIP_SPSTx10_Slide_9.78x27.58mm_W7.62mm_P2.54mm")
+      (reference "SW1") (unit 1) (value "SW_DIP_x10") (footprint "Button_Switch_THT:SW_DIP_SPSTx10_Piano_10.8x26.96mm_W7.62mm_P2.54mm")
     )
     (path "/30e0a99f-170f-40b8-b9a6-e5a266816a90"
