File: clock_logics/clock_logics.kicad_pcb (KiCad board)
At the start: 2 copper layers, 197 x 139 mm, 65 parts, among them J1 Conn_01x04_Male, J2 Conn_01x04_Male, J3 Conn_01x04_Male, U1 NE555P, U10 4017, U2 NE555P, U3 NE555P, U4 NE555P, U5 4011, U6 4001, U7 74HC240, U8 4020, U9 4076

Commit message: new schematics
Parts:
- added SW1: SW_DIP_x10, Button_Switch_THT:SW_DIP_SPSTx10_Piano_10.8x26.96mm_W7.62mm_P2.54mm, F.Cu at (46.1, 58.6)
- C11, C15, C3, C7: footprint Capacitor_THT:C_Disc_D5.0mm_W2.5mm_P2.50mm -> Capacitor_THT:C_Radial_D6.3mm_H11.0mm_P2.50mm
- J1, J2, J3: footprint Connector_PinSocket_2.54mm:PinSocket_1x04_P2.54mm_Vertical -> Connector_PinSocket_2.54mm:PinSocket_1x04_P2.54mm_Horizontal
- RV1, RV2, RV3, RV4, RV5, RV6, RV7, RV8: footprint Potentiometer_THT:Potentiometer_Bourns_3386C_Horizontal -> Potentiometer_THT:Potentiometer_Piher_PT-6-H_Horizontal
- moved C16 161.3 mm to (44.8, 107.0), turned to 90 degrees
- moved C4 160.7 mm to (56.8, 107.0), turned to 90 degrees
- moved C12 157.9 mm to (48.8, 107.0), turned to 90 degrees
- moved C8 157.2 mm to (52.8, 107.0), turned to 90 degrees
- moved C3 156.8 mm to (45.8, 92.0), turned to 90 degrees
- moved RV5 155.8 mm to (30.5, 57.8), turned to 0 degrees
- moved C7 155.2 mm to (45.8, 99.0), turned to 90 degrees
- moved RV7 154.9 mm to (30.5, 75.4), turned to 0 degrees
- moved RV4 153.8 mm to (30.5, 33.0), turned to 0 degrees
- moved RV2 153.0 mm to (30.5, 15.2), turned to 0 degrees
- moved RV6 151.0 mm to (30.5, 50.3), turned to 0 degrees
- moved RV8 150.8 mm to (30.5, 67.8), turned to 0 degrees
- moved C15 149.6 mm to (53.8, 92.0), turned to 90 degrees
- moved RV3 148.6 mm to (30.5, 40.6), turned to 0 degrees
- moved RV1 147.8 mm to (30.5, 22.9), turned to 0 degrees
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Connections:
- net Net-(C10-Pad2) renamed /ct3
- net Net-(C14-Pad2) renamed /ct4
- net Net-(C2-Pad2) renamed /ct1
- net Net-(C6-Pad2) renamed /ct2
- C11 pad 1: unconnected-(C11-Pad1) -> GND
- C11 pad 2: unconnected-(C11-Pad2) -> Net-(SW1-Pad16)
- C12 pad 1: unconnected-(C12-Pad1) -> GND
- C12 pad 2: unconnected-(C12-Pad2) -> Net-(SW1-Pad15)
- C15 pad 1: unconnected-(C15-Pad1) -> GND
- C15 pad 2: unconnected-(C15-Pad2) -> Net-(SW1-Pad14)
- C16 pad 1: unconnected-(C16-Pad1) -> GND
- C16 pad 2: unconnected-(C16-Pad2) -> Net-(SW1-Pad13)
- C3 pad 1: unconnected-(C3-Pad1) -> GND
- C3 pad 2: unconnected-(C3-Pad2) -> Net-(SW1-Pad20)
- C4 pad 1: unconnected-(C4-Pad1) -> GND
- C4 pad 2: unconnected-(C4-Pad2) -> Net-(SW1-Pad19)
- C7 pad 1: unconnected-(C7-Pad1) -> GND
- C7 pad 2: unconnected-(C7-Pad2) -> Net-(SW1-Pad18)
- C8 pad 1: unconnected-(C8-Pad1) -> GND
- C8 pad 2: unconnected-(C8-Pad2) -> Net-(C8-Pad2)
- J1 pad 3: unconnected-(J1-Pad3) -> /clk3out
- J1 pad 4: unconnected-(J1-Pad4) -> /clk4out
- R13 pad 2: /clk2out -> /clk4out
- R9 pad 2: /clk2out -> /clk3out
- U3 pad 3: /clk2out -> /clk3out
- U4 pad 3: /clk2out -> /clk4out
Routing:
- net +5V: track 0.00 -> 38.5 mm
- net /ct4: track 0.00 -> 36.9 mm
- net /ct3: track 0.00 -> 36.0 mm
- net /ct2: track 0.00 -> 35.0 mm
- net /ct1: track 0.00 -> 34.2 mm
- net GND: track 0.00 -> 16.0 mm
- net Net-(R10-Pad1): track 0.00 -> 13.4 mm
- net Net-(R14-Pad1): track 0.00 -> 12.2 mm
- net Net-(R2-Pad1): track 0.00 -> 12.1 mm
- net Net-(R6-Pad1): track 0.00 -> 11.7 mm
- net /clk4out: track 0.00 -> 6.78 mm
- net /clk1out: track 0.00 -> 5.39 mm
- net /clk3out: track 0.00 -> 5.37 mm
- net /clk2out: track 0.00 -> 5.37 mm
- net Net-(C13-Pad2): track 0.00 -> 4.67 mm
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Other:
- board outline removed
