File: sequencer/sequencer.kicad_pcb (KiCad board)
At the start: 2 copper layers, 42 x 110 mm, 24 parts, among them J1 PowerSupply, J2 Conn_01x06_Female, U1 LM741, U2 4020, U3 CD4051B

Commit message: SEQUENCER auto_saved_files
Parts:
- moved D2 109.3 mm to (117.0, 49.1), turned to 90 degrees
- moved D3 107.2 mm to (121.0, 52.1), turned to 90 degrees
- moved R1 106.9 mm to (144.0, 55.2), turned to -90 degrees
- moved U1 101.0 mm to (116.5, 77.8), turned to 180 degrees
- moved R3 97.5 mm to (121.0, 56.2), turned to -90 degrees
- moved D1 96.9 mm to (113.0, 46.1), turned to 90 degrees
- moved R5 85.8 mm to (113.0, 50.2), turned to -90 degrees
- moved R4 85.7 mm to (117.0, 52.2), turned to -90 degrees
- moved J2 55.7 mm to (138.3, 99.3)
- moved R2 54.4 mm to (116.5, 84.0), turned to 180 degrees
- moved C1 44.9 mm to (75.0, 86.0)
- moved U2 43.0 mm to (128.9, 42.1)
- moved U3 41.7 mm to (122.2, 72.1)
- moved C2 27.5 mm to (87.0, 88.0), turned to 90 degrees
- moved J1 23.1 mm to (127.7, 99.0), turned to -90 degrees
