File: relay_x8_12v/relay_x8_12v.kicad_pcb (KiCad board)
At the start: 2 copper layers, 114 x 146 mm, 35 parts, among them J1 Conn_01x12_Female, J2 Conn_01x12_Female, J3 Conn_01x12_Female, SW1 SW_SPDT, U1 ULN2803A

Commit message: relay kicad_pcb
Parts:
- moved RL8 97.7 mm to (64.0, 75.0)
- moved D8 74.0 mm to (43.0, 85.0)
- moved R8 74.0 mm to (48.0, 87.8)
- moved D5 72.0 mm to (43.0, 158.0)
- moved R5 72.0 mm to (48.0, 160.8)
- moved RL7 69.7 mm to (64.0, 89.0)
- moved RL1 56.0 mm to (64.0, 130.7)
- moved RL2 56.0 mm to (64.0, 144.7)
- moved RL3 56.0 mm to (64.0, 158.7)
- moved RL4 56.0 mm to (64.0, 172.7)
- moved RL6 41.7 mm to (64.0, 103.0)
- moved D7 25.8 mm to (43.0, 109.2)
- moved R7 25.8 mm to (48.0, 112.0)
- moved R6 22.0 mm to (48.0, 135.8)
- moved D6 22.0 mm to (43.0, 133.5)
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Routing:
- net /power_on: track 364.3 -> 0.00 mm
- net /x5: track 123.2 -> 0.00 mm
- net /o8: track 117.5 -> 0.00 mm
- net /o4: track 112.1 -> 0.00 mm
- net /c5: track 106.9 -> 0.00 mm
- net /y5: track 104.2 -> 0.00 mm
- net /o7: track 98.4 -> 0.00 mm
- net /o3: track 90.7 -> 0.00 mm
- net /y6: track 86.0 -> 0.00 mm
- net /o6: track 85.1 -> 0.00 mm
- net /x6: track 84.6 -> 0.00 mm
- net /c6: track 84.3 -> 0.00 mm
- net /y7: track 81.7 -> 0.00 mm
- net /c7: track 79.6 -> 0.00 mm
- net /y8: track 77.4 -> 0.00 mm
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Other:
- board size 114 x 146 mm -> 112 x 146 mm
